File: gmap4real_teensy/porti2c.sch (KiCad schematic (older format))
At the start: 1 part

Commit message: teensy: simplify (no agnd to buttons, no agnd to i2c port)
Parts:
- porti2c0: value Conn_01x05 -> Conn_01x04; footprint Connector_PinHeader_2.54mm:PinHeader_1x05_P2.54mm_Vertical -> Connector_PinHeader_2.54mm:PinHeader_1x04_P2.54mm_Vertical; symbol Connector_Generic:Conn_01x05 -> Connector_Generic:Conn_01x04
Connections:
- net agnd is gone; now on net 3.3v: porti2c0.2 (Pin_2)
- net 3.3v: no longer porti2c0.3 (Pin_3)
- net i2cscl0: now also porti2c0.3 (Pin_3); no longer porti2c0.4 (Pin_4)
- net i2csda0: now also porti2c0.4 (Pin_4); no longer porti2c0.5 (Pin_5)
Changed lines of the file:
@@
 Text GLabel 7050 3300 0    50   Input ~ 0
 gnd
+Text GLabel 7050 3400 0    50   Input ~ 0
+3.3v
 Text GLabel 7050 3500 0    50   Input ~ 0
-3.3v
+i2cscl0
 Text GLabel 7050 3600 0    50   Input ~ 0
-i2cscl0
-Text GLabel 7050 3700 0    50   Input ~ 0
 i2csda0
-Text GLabel 7050 3400 0    50   Input ~ 0
-agnd
 $Comp
-L Connector_Generic:Conn_01x05 porti2c0
+L Connector_Generic:Conn_01x04 porti2c0
 U 1 1 5CA4A24A
-P 7250 3500
-F 0 "porti2c0" H 7330 3542 50  0000 L CNN
-F 1 "Conn_01x05" H 7330 3451 50  0000 L CNN
-F 2 "Connector_PinHeader_2.54mm:PinHeader_1x05_P2.54mm_Vertical" H 7250 3500 50  0001 C CNN
-F 3 "~" H 7250 3500 50  0001 C CNN
-	1    7250 3500
+P 7250 3400
+F 0 "porti2c0" H 7330 3442 50  0000 L CNN
+F 1 "Conn_01x04" H 7330 3351 50  0000 L CNN
+F 2 "Connector_PinHeader_2.54mm:PinHeader_1x04_P2.54mm_Vertical" H 7250 3400 50  0001 C CNN
+F 3 "~" H 7250 3400 50  0001 C CNN
+	1    7250 3400
 	1    0    0    -1
 $EndComp
